Commit message: Add an end-effector to the model and forward kinematics node

File: src/robot_arm_description/urdf/robot_arm.urdf (robot description, URDF)
Before this commit: robot robot_arm, 3 links, 2 joints
Links:
- added link end_effector; visual sphere radius=0.04
Joints:
- added joint end_effector_joint: type fixed, parent forearm, child end_effector, origin xyz=0 0 0.4
